File: pcb/bigbro_box/display.kicad_sch (KiCad schematic)
At the start: 18 parts, among them J5 Conn_01x24_MountingPin, Q3 Si1308EDL

Commit message: Widened isolation slot
Parts:
- J5: value Conn_01x24_MountingPin -> 2-1734839-4
- Q3: footprint Package_TO_SOT_SMD:SOT-23_Handsoldering -> Package_TO_SOT_SMD:SOT-323_SC-70_Handsoldering
Connections:
- net GND: now also J5.MP (MountPin)
- no-connect marks 4 -> 3
Changed lines of the file:
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@@
   (no_connect (at 176.53 53.34))
   (no_connect (at 176.53 91.44))
-  (no_connect (at 181.61 109.22))
   (wire (pts (xy 85.09 90.17) (xy 100.33 90.17))
     (stroke (width 0) (type default) (color 0 0 0 0))
@@
   )
   (wire (pts (xy 175.26 111.76) (xy 175.26 113.03))
+    (stroke (width 0) (type default) (color 0 0 0 0))
+  )
+  (wire (pts (xy 175.26 111.76) (xy 181.61 111.76))
+    (stroke (width 0) (type default) (color 0 0 0 0))
+  )
+  (wire (pts (xy 181.61 111.76) (xy 181.61 109.22))
     (stroke (width 0) (type default) (color 0 0 0 0))
   )
@@
       (effects (font (size 1.27 1.27)) (justify left))
     )
-    (property "Footprint" "Package_TO_SOT_SMD:SOT-23_Handsoldering" (id 2) (at 114.3 93.98 0)
+    (property "Footprint" "Package_TO_SOT_SMD:SOT-323_SC-70_Handsoldering" (id 2) (at 114.3 93.98 0)
       (effects (font (size 1.27 1.27)) hide)
     )
@@
       (effects (font (size 1.27 1.27)) (justify left))
     )
-    (property "Value" "Conn_01x24_MountingPin" (id 1) (at 184.15 78.0414 0)
-      (effects (font (size 1.27 1.27)) (justify left))
-    )
+    (property "Value" "2-1734839-4" (id 1) (at 184.15 78.0414 0)
+      (effects (font (size 1.27 1.27)) (justify left))
+    )

Commit message: Order1
Parts:
- J5: MPN (none) -> GDEY0213Z98
Changed lines of the file:
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@@
       (effects (font (size 1.27 1.27)) hide)
     )
-    (property "Datasheet" "~" (id 3) (at 181.61 73.66 0)
+    (property "Datasheet" "https://v4.cecdn.yun300.cn/100001_1909185148/GDEY0213Z98.pdf" (id 3) (at 181.61 73.66 0)
       (effects (font (size 1.27 1.27)) hide)
     )
+    (property "MPN" "GDEY0213Z98" (id 4) (at 181.61 73.66 0)
+      (effects (font (size 1.27 1.27)) hide)
+    )
