File: pcb/bigbro_box_v2/bigbro_box.kicad_sch (KiCad schematic)
At the start: 46 parts, among them J1 Current Sense, J2 Display, J3 Mains, J4 Debug, J5 RFID, J6 Relay, J7 Ext, K1 G5LE-1, Q1 MMBT3904, Q2 MMBT3904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

Commit message: Flip display connector.
Parts:
- J2: footprint Connector_PinHeader_2.54mm:PinHeader_1x08_P2.54mm_Vertical -> Connector_PinSocket_2.54mm:PinSocket_1x08_P2.54mm_Vertical
Changed lines of the file:
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@@
       (effects (font (size 1.27 1.27)) (justify left))
     )
-    (property "Footprint" "Connector_PinHeader_2.54mm:PinHeader_1x08_P2.54mm_Vertical" (at 139.7 66.04 0)
+    (property "Footprint" "Connector_PinSocket_2.54mm:PinSocket_1x08_P2.54mm_Vertical" (at 139.7 66.04 0)
       (effects (font (size 1.27 1.27)) hide)
     )

Commit message: Forgot to save
Parts:
- Q3: symbol Device:Q_NMOS_GDS -> Device:Q_NMOS_GSD
Connections:
- net GND: now also Q3.2 (S); no longer Q3.3 (S)
- net at D1.2 (A), K1.2, R6.2: now also Q3.3 (D); no longer Q3.2 (D)
Changed lines of the file:
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@@
     )
   )
-  (symbol (lib_id "Device:Q_NMOS_GDS") (at 339.09 101.6 0) (unit 1)
+  (symbol (lib_id "Device:Q_NMOS_GSD") (at 339.09 101.6 0) (unit 1)
     (in_bom yes) (on_board yes) (dnp no) (fields_autoplaced)
     (property "Reference" "Q3" (at 345.44 100.965 0)
