File: pcb/bigbro_box_v2/bigbro_box.kicad_sch (KiCad schematic)
At the start: 46 parts, among them J1 Current Sense, J2 Display, J3 Mains, J4 Debug, J5 RFID, J6 Relay, J7 Ext, K1 G5LE-1, Q1 MMBT3904, Q2 MMBT3904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

Commit message: Fix Q3 footprint, Q4 resistor values.
Parts:
- C1: value 1uF -> 1u
- C2: value 10uF -> 10u
- Q3: footprint Package_TO_SOT_SMD:SOT-323_SC-70 -> Package_TO_SOT_SMD:SOT-23
- R1: value 1k -> 4k7
- R2: value 10k -> 1k
Changed lines of the file:
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@@
   (symbol (lib_id "Device:C_Small") (at 387.35 43.18 0) (unit 1)
     (in_bom yes) (on_board yes) (dnp no) (fields_autoplaced)
-    (property "Reference" "C2" (at 389.89 41.9099 0)
-      (effects (font (size 1.27 1.27)) (justify left))
-    )
-    (property "Value" "10uF" (at 389.89 44.4499 0)
+    (property "Reference" "C2" (at 389.89 42.5513 0)
+      (effects (font (size 1.27 1.27)) (justify left))
+    )
+    (property "Value" "10u" (at 389.89 45.0913 0)
       (effects (font (size 1.27 1.27)) (justify left))
     )
@@
       (effects (font (size 1.27 1.27)) (justify left))
     )
-    (property "Footprint" "Package_TO_SOT_SMD:SOT-323_SC-70" (at 344.17 99.06 0)
+    (property "Footprint" "Package_TO_SOT_SMD:SOT-23" (at 344.17 99.06 0)
       (effects (font (size 1.27 1.27)) hide)
     )
@@
       (effects (font (size 1.27 1.27)) (justify right))
     )
-    (property "Value" "10k" (at 71.12 168.9099 0)
+    (property "Value" "1k" (at 71.12 168.9099 0)
       (effects (font (size 1.27 1.27)) (justify right))
     )
@@
       (effects (font (size 1.27 1.27)) (justify right))
     )
-    (property "Value" "1k" (at 67.3101 170.18 0)
+    (property "Value" "4k7" (at 67.3101 170.18 0)
       (effects (font (size 1.27 1.27)) (justify right))
     )
@@
       (effects (font (size 1.27 1.27)) (justify left))
     )
-    (property "Value" "1uF" (at 364.49 44.4499 0)
-      (effects (font (size 1.27 1.27)) (justify left))
-    )
+    (property "Value" "1u" (at 364.49 44.4499 0)
+      (effects (font (size 1.27 1.27)) (justify left))
+    )
