File: pcb/bigbro_box.kicad_sch (KiCad schematic)
At the start: 46 parts, among them J1 Current Sense, J2 Display, J3 Mains, J4 Debug, J5 RFID, J6 Relay, J7 Ext, K1 G5LE-1, Q1 MMBT3904, Q2 MMBT3904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

Commit message: Move.
Connections:
- net ESP_RFID_TX: now also R10.1, R11.2; no longer R11.1
- new net: R11.1, U5.6 (TX)
Other:
- moved on the sheet: R10, R11
Changed lines of the file:
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@@
   (junction (at 387.35 39.37) (diameter 0) (color 0 0 0 0)
   )
+  (junction (at 198.12 48.26) (diameter 0) (color 0 0 0 0)
+  )
   (junction (at 356.87 39.37) (diameter 0) (color 0 0 0 0)
   )
@@
   )
   (junction (at 24.13 92.71) (diameter 0) (color 0 0 0 0)
-  )
-  (junction (at 198.12 40.64) (diameter 0) (color 0 0 0 0)
   )
   (junction (at 35.56 121.92) (diameter 0) (color 0 0 0 0)
@@
     (stroke (width 0) (type default))
   )
+  (wire (pts (xy 198.12 48.26) (xy 198.12 49.53))
+    (stroke (width 0) (type default))
+  )
   (wire (pts (xy 33.02 87.63) (xy 35.56 85.09))
     (stroke (width 0) (type default))
@@
     (stroke (width 0) (type default))
   )
+  (wire (pts (xy 165.1 81.28) (xy 167.64 81.28))
+    (stroke (width 0) (type default))
+  )
+  (wire (pts (xy 167.64 81.28) (xy 167.64 86.36))
+    (stroke (width 0) (type default))
+  )
+  (wire (pts (xy 128.27 142.24) (xy 127 142.24))
+    (stroke (width 0) (type default))
+  )
+  (wire (pts (xy 129.54 71.12) (xy 129.54 77.47))
+    (stroke (width 0) (type default))
+  )
+  (wire (pts (xy 167.64 57.15) (xy 179.07 57.15))
+    (stroke (width 0) (type default))
+  )
+  (wire (pts (xy 179.07 21.59) (xy 179.07 25.4))
+    (stroke (width 0) (type default))
+  )
+  (wire (pts (xy 35.56 86.36) (xy 35.56 87.63))
+    (stroke (width 0) (type default))
+  )
+  (wire (pts (xy 181.61 29.21) (xy 181.61 25.4))
+    (stroke (width 0) (type default))
+  )
+  (wire (pts (xy 149.86 147.32) (xy 149.86 148.59))
+    (stroke (width 0) (type default))
+  )
+  (wire (pts (xy 325.12 101.6) (xy 325.12 102.87))
+    (stroke (width 0) (type default))
+  )
+  (wire (pts (xy 331.47 101.6) (xy 334.01 101.6))
+    (stroke (width 0) (type default))
+  )
   (wire (pts (xy 190.5 40.64) (xy 198.12 40.64))
     (stroke (width 0) (type default))
   )
-  (wire (pts (xy 165.1 81.28) (xy 167.64 81.28))
-    (stroke (width 0) (type default))
-  )
-  (wire (pts (xy 167.64 81.28) (xy 167.64 86.36))
-    (stroke (width 0) (type default))
-  )
-  (wire (pts (xy 128.27 142.24) (xy 127 142.24))
-    (stroke (width 0) (type default))
-  )
-  (wire (pts (xy 129.54 71.12) (xy 129.54 77.47))
-    (stroke (width 0) (type default))
-  )
-  (wire (pts (xy 167.64 57.15) (xy 179.07 57.15))
-    (stroke (width 0) (type default))
-  )
-  (wire (pts (xy 179.07 21.59) (xy 179.07 25.4))
-    (stroke (width 0) (type default))
-  )
-  (wire (pts (xy 35.56 86.36) (xy 35.56 87.63))
-    (stroke (width 0) (type default))
-  )
-  (wire (pts (xy 181.61 29.21) (xy 181.61 25.4))
-    (stroke (width 0) (type default))
-  )
-  (wire (pts (xy 149.86 147.32) (xy 149.86 148.59))
-    (stroke (width 0) (type default))
-  )
-  (wire (pts (xy 325.12 101.6) (xy 325.12 102.87))
-    (stroke (width 0) (type default))
-  )
-  (wire (pts (xy 331.47 101.6) (xy 334.01 101.6))
-    (stroke (width 0) (type default))
-  )
   (wire (pts (xy 88.9 69.85) (xy 93.98 69.85))
     (stroke (width 0) (type default))
@@
     (stroke (width 0) (type default))
   )
-  (wire (pts (xy 198.12 40.64) (xy 198.12 39.37))
-    (stroke (width 0) (type default))
-  )
   (wire (pts (xy 55.88 29.21) (xy 58.42 29.21))
     (stroke (width 0) (type default))
@@
     (stroke (width 0) (type default))
   )
-  (wire (pts (xy 198.12 29.21) (xy 198.12 31.75))
-    (stroke (width 0) (type default))
-  )
   (wire (pts (xy 165.1 40.64) (xy 170.18 40.64))
     (stroke (width 0) (type default))
@@
     (stroke (width 0) (type default))
   )
-  (wire (pts (xy 198.12 40.64) (xy 198.12 41.91))
-    (stroke (width 0) (type default))
-  )
   (wire (pts (xy 25.4 173.99) (xy 25.4 177.8))
     (stroke (width 0) (type default))
@@
     (stroke (width 0) (type default))
   )
-  (wire (pts (xy 198.12 57.15) (xy 198.12 49.53))
-    (stroke (width 0) (type default))
-  )
   (wire (pts (xy 134.62 212.09) (xy 132.08 212.09))
     (stroke (width 0) (type default))
@@
     (stroke (width 0) (type default))
   )
+  (wire (pts (xy 198.12 48.26) (xy 205.74 48.26))
+    (stroke (width 0) (type default))
+  )
   (wire (pts (xy 355.6 44.45) (xy 356.87 44.45))
     (stroke (width 0) (type default))
@@
   )
   (wire (pts (xy 76.2 175.26) (xy 77.47 175.26))
-    (stroke (width 0) (type default))
-  )
-  (wire (pts (xy 200.66 29.21) (xy 198.12 29.21))
     (stroke (width 0) (type default))
   )
@@
     )
   )
-  (global_label "ESP_RFID_TX" (shape input) (at 200.66 29.21 0) (fields_autoplaced)
+  (global_label "ESP_RFID_TX" (shape input) (at 205.74 48.26 0) (fields_autoplaced)
     (effects (font (size 1.27 1.27)) (justify left))
-    (property "Intersheetrefs" "${INTERSHEET_REFS}" (at 215.0474 29.1306 0)
+    (property "Intersheetrefs" "${INTERSHEET_REFS}" (at 220.1274 48.1806 0)
       (effects (font (size 1.27 1.27)) (justify left) hide)
     )
@@
     )
   )
-  (symbol (lib_id "Device:R") (at 198.12 45.72 0) (unit 1)
-    (in_bom yes) (on_board yes) (dnp no) (fields_autoplaced)
-    (property "Reference" "R10" (at 200.66 45.085 0)
-      (effects (font (size 1.27 1.27)) (justify left))
-    )
-    (property "Value" "2k2" (at 200.66 47.625 0)
-      (effects (font (size 1.27 1.27)) (justify left))
-    )
-    (property "Footprint" "Resistor_SMD:R_0603_1608Metric" (at 196.342 45.72 90)
-      (effects (font (size 1.27 1.27)) hide)
-    )
-    (property "Datasheet" "~" (at 198.12 45.72 0)
+  (symbol (lib_id "Device:R") (at 198.12 53.34 0) (unit 1)
+    (in_bom yes) (on_board yes) (dnp no) (fields_autoplaced)
+    (property "Reference" "R10" (at 200.66 52.705 0)
+      (effects (font (size 1.27 1.27)) (justify left))
+    )
+    (property "Value" "2k2" (at 200.66 55.245 0)
+      (effects (font (size 1.27 1.27)) (justify left))
+    )
+    (property "Footprint" "Resistor_SMD:R_0603_1608Metric" (at 196.342 53.34 90)
+      (effects (font (size 1.27 1.27)) hide)
+    )
+    (property "Datasheet" "~" (at 198.12 53.34 0)
       (effects (font (size 1.27 1.27)) hide)
     )
@@
     )
   )
-  (symbol (lib_id "Device:R") (at 198.12 35.56 0) (unit 1)
-    (in_bom yes) (on_board yes) (dnp no) (fields_autoplaced)
-    (property "Reference" "R11" (at 200.66 34.925 0)
-      (effects (font (size 1.27 1.27)) (justify left))
-    )
-    (property "Value" "1k2" (at 200.66 37.465 0)
-      (effects (font (size 1.27 1.27)) (justify left))
-    )
-    (property "Footprint" "Resistor_SMD:R_0603_1608Metric" (at 196.342 35.56 90)
-      (effects (font (size 1.27 1.27)) hide)
-    )
-    (property "Datasheet" "~" (at 198.12 35.56 0)
-      (effects (font (size 1.27 1.27)) hide)
-    )
+  (symbol (lib_id "Device:R") (at 198.12 44.45 0) (unit 1)
+    (in_bom yes) (on_board yes) (dnp no) (fields_autoplaced)
+    (property "Reference" "R11" (at 200.66 43.815 0)
+      (effects (font (size 1.27 1.27)) (justify left))
+    )
+    (property "Value" "1k2" (at 200.66 46.355 0)
+      (effects (font (size 1.27 1.27)) (justify left))
+    )
+    (property "Footprint" "Resistor_SMD:R_0603_1608Metric" (at 196.342 44.45 90)
+      (effects (font (size 1.27 1.27)) hide)
+    )
+    (property "Datasheet" "~" (at 198.12 44.45 0)
+      (effects (font (size 1.27 1.27)) hide)
+    )
